File: Hardware/CommandCenter_KICAD/Audio.sch (KiCad schematic (older format))
At the start: 16 parts

Commit message: Layout started
Parts:
- removed J?: SPKR0-, NFC_Toy_Lib:Pad_SMD_Small, symbol Pad:Pad
- removed J?: SPKR0+, NFC_Toy_Lib:Pad_SMD_Small, symbol Pad:Pad
- removed J?: SPKR1-, NFC_Toy_Lib:Pad_SMD_Small, symbol Pad:Pad
- removed J?: SPKR1+, NFC_Toy_Lib:Pad_SMD_Small, symbol Pad:Pad
- added J6: SPKR0, Connector_PinHeader_2.54mm:PinHeader_1x02_P2.54mm_Vertical, symbol Connector_Generic:Conn_01x02
- added J7: SPKR1, Connector_PinHeader_2.54mm:PinHeader_1x02_P2.54mm_Vertical, symbol Connector_Generic:Conn_01x02
- C13, C14, C15: renamed from C?; footprint Capacitors_SMD:C_0402 -> Capacitor_SMD:C_0603_1608Metric_Pad1.05x0.95mm_HandSolder
- C16, C17: renamed from C?; footprint Capacitors_SMD:C_0603_HandSoldering -> Capacitor_SMD:C_0603_1608Metric_Pad1.05x0.95mm_HandSolder
- J5: renamed from J?; footprint MOLEX_503182-1852 -> CommandCenter:MOLEX_503182-1852
- R15, R16, R17, R18: renamed from R?; footprint Resistors_SMD:R_0603_HandSoldering -> Resistor_SMD:R_0603_1608Metric_Pad1.05x0.95mm_HandSolder
- U4, U5: renamed from U?; footprint NFC_Toy_Lib:QFN50P300X300X80-17N -> CommandCenter:QFN50P300X300X80-17N
Connections:
- net at U4.10 (OUTN): now also J6.1 (Pin_1)
- net at U4.9 (OUTP): now also J6.2 (Pin_2)
- net at U5.10 (OUTN): now also J7.1 (Pin_1)
- net at U5.9 (OUTP): now also J7.2 (Pin_2)
