File: Hardware/CommandCenter_KICAD/BarGraph.sch (KiCad schematic (older format))
At the start: 12 parts

Commit message: Layout started
Parts:
- C46, C47, C48: renamed from C?; footprint Capacitors_SMD:C_0402 -> Capacitor_SMD:C_0603_1608Metric_Pad1.05x0.95mm_HandSolder
- R47, R48, R49: renamed from R?; footprint (none) -> Resistor_SMD:R_0603_1608Metric_Pad1.05x0.95mm_HandSolder
- U29: renamed from U?; footprint (none) -> Package_SO:SOIC-24W_7.5x15.4mm_P1.27mm
- gave numbers to parts that had none: 5
Connections:
- net GND: now also U30.7 (GND)
- net SEG_C: no longer BAR1.1 (A), BAR1.2 (A), BAR1.3 (A), BAR1.4 (A), BAR1.5 (A), BAR1.6 (A), BAR1.7 (A), BAR1.8 (A)
- net SEG_D: now also BAR1.1 (A), BAR1.2 (A), BAR1.3 (A), BAR1.4 (A), BAR1.5 (A), BAR1.6 (A), BAR1.7 (A), BAR1.8 (A)
- net BG_MOSI_ renamed BG_SPI_MOSI
- net BG_MOSI_5V renamed BG_SPI_MOSI_5V
- net BG_SCK renamed BG_SPI_SCK
- net BG_SCK_5V renamed BG_SPI_SCK_5V
- net BG_SS renamed BG_SPI_SS
- net BG_SS_5V renamed BG_SPI_SS_5V
Other:
- moved on the sheet: C48
