File: Hardware/CommandCenter_KICAD/DotStar.sch (KiCad schematic (older format))
At the start: 37 parts

Commit message: Layout started
Parts:
- added C30, C35, C40, C45: 0.1u, Capacitor_SMD:C_0603_1608Metric_Pad1.05x0.95mm_HandSolder, symbol Device:C
- added U25, U26, U27, U28: APA102, CommandCenter:APA102_hand_solder, symbol APA102:APA102
- C24, C25, C26, C27, C28, C29, C31, C32, C33, C34, C36, C37, C38, C39, C41, C42, C43, C44: renamed from C?; footprint Capacitors_SMD:C_0402 -> Capacitor_SMD:C_0603_1608Metric_Pad1.05x0.95mm_HandSolder
- TP8, TP9: renamed from TP?; footprint (none) -> TestPoint:TestPoint_Pad_2.0x2.0mm
- U10, U11, U12, U14, U15, U16, U17, U18, U19, U20, U21, U22, U23, U24, U8, U9: renamed from U?; footprint NFC_Toy_Lib:APA102_hand_solder -> CommandCenter:APA102_hand_solder
- U13: renamed from U?; footprint NFC_Toy_Lib:SOP50P310X90-8N -> CommandCenter:SOP50P310X90-8N
Connections:
- net +5V: now also C30.1, C35.1, C40.1, C45.1, U25.4 (VCC), U26.4 (VCC), U27.4 (VCC), U28.4 (VCC)
- net GND: now also C30.2, C35.2, C40.2, C45.2, U25.3 (GND), U26.3 (GND), U27.3 (GND), U28.3 (GND)
- net DotStar_CO_3: now reaches U24.5 (CO)
- net DotStar_CO_3: now also U25.2 (CI)
- net DotStar_DO_3: now reaches U24.6 (DO)
- net DotStar_DO_3: now also U25.1 (DI)
- new net: U25.5 (CO), U26.2 (CI)
- new net: U25.6 (DO), U26.1 (DI)
- new net: U26.5 (CO), U27.2 (CI)
- new net: U26.6 (DO), U27.1 (DI)
- new net: U27.5 (CO), U28.2 (CI)
- new net: U27.6 (DO), U28.1 (DI)
Other:
- moved on the sheet: C26, C27, C28, C29, C31, C32, C33, C34, C36, C37, C38, C39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
