File: Hardware/CommandCenter_KICAD/CommandCenter_KICAD.kicad_pcb (KiCad board)
At the start: 2 copper layers, 171 parts, among them J1 Battery, J10 LED2, J11 LED3, J12 Wake, J13 SW0, J14 SW1, J15 SW2, J16 SW3, J17 JLink_Mini, J18 Bar Graph SW, J2 Motor_Switches, J3 JLink_Mini, J4 Motor, J5 503182-1852, J6 SPKR0, J7 SPKR1, J8 LED0, J9 LED1, Q1 DMG1012T-7, Q2 DMG1012T-7, Q3 DMG1012T-7, Q4 DMG1012T-7, Q5 DMG1012T-7, Q6 DMG1012T-7, U1 TPS61032, U10 APA102, U11 APA102, U12 APA102, U13 SN74LVC2T45, U14 APA102, U15 APA102, U16 APA102, U17 APA102, U18 APA102, U19 APA102, U2 STM32L0-LQFP48, U20 APA102, U21 APA102, U22 APA102, U23 APA102, U24 APA102, U25 APA102, U26 APA102, U27 APA102, U28 APA102, U29 MAX7219, U3 MIC5225, U30 TXB0104PW, U4 MAX98357, U5 MAX98357, U6 STM32L0-LQFP48, U7 APDS-9960, U8 APA102, U9 APA102

Commit message: Light Project Stable
DotStars and bar graph working. Getting master read nack on I2C to color sensor.
Parts:
- removed C18, C4: 0.1u, Capacitor_SMD:C_0603_1608Metric_Pad1.05x0.95mm_HandSolder
- BAR1, BAR2, BAR3, BAR4, C26, C27, C28, C29, C30, C31, C32, C33, C34, C35, C36, C37, C38, C39, C40, C41, C42, C43, C44, C45, U10, U11, U12, U14, U15, U16, U17, U18, U19, U20, U21, U22, U23, U24, U25, U26, U27, U28, U7, U8, U9: moved to B.Cu
- J3, J5, U2: moved to F.Cu
- moved TP8 165.7 mm to (187.7, 82.5)
- moved C14 165.1 mm to (188.1, 43.1)
- moved R40 162.9 mm to (181.4, 27.6), turned to 270 degrees
- moved C16 162.5 mm to (188.1, 40.1)
- moved TP9 160.8 mm to (177.5, 82.5)
- moved R16 158.9 mm to (185.3, 51.6)
- moved R29 158.6 mm to (235.7, 63.8), turned to 90 degrees
- moved C39 157.3 mm to (130.6, 37.8), turned to 180 degrees
- moved C13 156.5 mm to (134.0, 33.4), turned to 180 degrees
- moved R45 156.2 mm to (174.4, 23.1), turned to 180 degrees
- moved R48 155.8 mm to (178.7, 148.3), turned to 180 degrees
- moved C35 155.3 mm to (159.5, 52.6), turned to 180 degrees
- moved C15 151.2 mm to (106.4, 31.2), turned to 270 degrees
- moved TP7 150.7 mm to (168.1, 38.1)
- moved C40 150.7 mm to (158.8, 66.8), turned to 90 degrees
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- renumbered MK4 to MKe
Connections:
- R42 pad 1: Net-(R42-Pad1) -> +3V3
- R43 pad 1: Net-(R42-Pad1) -> +3V3
- R44 pad 1: Net-(R42-Pad1) -> +3V3
- R46 pad 1: Net-(R42-Pad1) -> +3V3
Routing:
- net +3V3: track 0.00 -> 843.9 mm, vias 0 -> 43
- net +5V: track 0.00 -> 720.2 mm, vias 0 -> 12
- net GND: track 0.00 -> 424.3 mm, vias 0 -> 112
- net WKUP: track 0.00 -> 283.1 mm, vias 0 -> 6
- net AUDIO_UART_RX: track 0.00 -> 231.4 mm, vias 0 -> 6
- net AUDIO_UART_TX: track 0.00 -> 221.6 mm, vias 0 -> 6
- net nRST_LIGHT: track 0.00 -> 218.5 mm, vias 0 -> 7
- net SEG_C: track 0.00 -> 167.1 mm, vias 0 -> 2
- net DotStar_Clk_3V: track 0.00 -> 164.0 mm, vias 0 -> 2
- net DotStar_Data_3V: track 0.00 -> 158.5 mm
- net SWDIO_LIGHT: track 0.00 -> 141.8 mm, vias 0 -> 2
- net SEG_D: track 0.00 -> 141.6 mm, vias 0 -> 1
- net SWCLK_LIGHT: track 0.00 -> 140.0 mm, vias 0 -> 1
- net I2S_CK: track 0.00 -> 135.0 mm, vias 0 -> 2
- net I2S_SD: track 0.00 -> 133.9 mm, vias 0 -> 5
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- added copper zone on B.Cu, net GND
- added copper zone on F.Cu, net GND
Other:
- board outline added: 176 x 145 mm
- net class Default: clearance 0.2 -> 0.13
- net class Power added: clearance 0.13, trace_width 0.5, via_dia 0.8, via_drill 0.4
- rule trace_clearance: 0.2 -> 0.13
- board text added: "+"
- board text added: "-"
- board text added: "Audio SWD"
- board text added: "BAR GRAPH SWITCHES"
- board text added: "Command Center"
- board text added: "DOTSTAR_CLK"
- board text added: "DOTSTAR_DATA"
- board text added: "I2S_CK"
- board text added: "I2S_DATA"
- board text added: "I2S_LRCK"
- board text added: "LED0"
- board text added: "LED1"
- board text added: "LED2"
- board text added: "LED3"
- board text added: "Lights SWD"
- board text added: "MOTOR"
- board text added: "MOTOR SWITCHES"
- board text added: "Rev 1.0 AC"
- board text added: "SD MISO"
- board text added: "SD MOSI"
- board text added: "SD NSS"
- board text added: "SD SCK"
- board text added: "SPKR0"
- board text added: "SPRK1"
- board text added: "SW0"
- board text added: "SW1"
- board text added: "SW2"
- board text added: "SW3"
- board text added: "WKUP"
